File: Drone_1.kicad_sch (KiCad schematic)
At the start: 6 parts, among them J1 ESP-32_DevkitC, U1 E, U2 MPU6050, U3 GY-NEO6MV2, U4 BME280, U5 HMC5883L

Commit message: Add files via upload
Parts:
- added U6, U7: mp1584, symbol mp1584:mp1584m
- added U8: Flysky fs-a8s, symbol flysky fs-a8s:Flysky_fs-a8s
Connections:
- net +3.3V: now also J1.15 (Pin_15), U4.1 (VCC), U4.5 (CSB), U5.1 (VCC), U6.1 (OUT+); no longer J1.16 (Pin_16)
- net +5V: now also U7.1 (OUT+), U8.2 (VCC); no longer J1.15 (Pin_15)
- net 0: now also U4.2 (GND), U5.2 (GND), U6.4 (OUT-), U7.4 (OUT-), U8.1 (GND); no longer J1.17 (Pin_17)
- net at U4.3 (SCL): now also J1.2 (Pin_2)
- net at U4.4 (SDA): now also J1.3 (Pin_3)
- net at J1.21 (Pin_21): now also U8.3 (SBUS)
- net at J1.4 (Pin_4): now also U5.4 (SDA)
- net at J1.5 (Pin_5): now also U5.3 (SCL)
- no-connect marks 3 -> 5
Other:
- moved on the sheet: U1, U4, U5
