File: OLD/Drone_1.kicad_pcb (KiCad board)
At the start: 4 copper layers, 100 x 120 mm, 25 parts, among them J1 ESP-32_DevkitC, J2 Conn_01x08_Pin, U1 Rasberry Pi 0W, U10 Bidirectional ESC, U2 MPU6050, U3 GY-NEO6MV2, U4 BME280, U5 HMC5883L, U6 mp1584, U7 mp1584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

Commit message: welcome
Parts:
- removed U9: Bidirectional ESC, Bidirectional_ESC:Bi_ESC_foot
- U10: value Bidirectional ESC -> ~; footprint Bidirectional_ESC:Bi_ESC_foot -> 4x1_ESC:4x1_ESC
- moved U10 93.3 mm to (149.1, 89.8)
- moved J2 0.91 mm to (66.4, 109.7)
- moved U2 0.69 mm to (137.5, 72.4)
Connections:
- J1 pad 12: unconnected-(J1-Pin_12-Pad12) -> Net-(J1-Pin_12)
- J1 pad 18: Net-(J1-Pin_18) -> unconnected-(J1-Pin_18-Pad18)
- J1 pad 19: Net-(J1-Pin_19) -> unconnected-(J1-Pin_19-Pad19)
- J1 pad 9: unconnected-(J1-Pin_9-Pad9) -> Net-(J1-Pin_9)
Routing:
- net Net-(J1-Pin_10): track 113.8 -> 0.00 mm
- net Net-(J1-Pin_11): track 110.4 -> 0.00 mm
- net Net-(J1-Pin_19): track 25.0 -> 0.00 mm
- net Net-(J1-Pin_18): track 21.6 -> 0.00 mm
- net 0: track 41.2 -> 24.4 mm, vias 7 -> 5
- net +7.5V: track 4.77 -> 17.1 mm
- net GND: track 0.00 -> 11.6 mm, vias 0 -> 1
- net Net-(J1-Pin_29): track 40.6 -> 48.8 mm
- net Net-(J1-Pin_21): track 32.3 -> 26.5 mm
- net Net-(J1-Pin_30): track 50.2 -> 44.8 mm
- net Net-(J1-Pin_28): track 41.4 -> 39.5 mm
- net Net-(J1-Pin_20): track 73.7 -> 74.7 mm
- net Net-(J1-Pin_23): track 64.6 -> 65.4 mm
- net Net-(J1-Pin_22): track 66.8 -> 67.7 mm
- net +5V: track 6.77 -> 7.48 mm
