File: OLD/Drone_1.kicad_sch (KiCad schematic)
At the start: 9 parts, among them J1 ESP-32_DevkitC, U1 E, U2 MPU6050, U3 GY-NEO6MV2, U4 BME280, U5 HMC5883L, U6 mp1584, U7 mp1584, U8 Flysky fs-a8s

Commit message: welcome
Parts:
- added BT1: Battery, Connector_JST:JST_EH_S2B-EH_1x02_P2.50mm_Horizontal, symbol Device:Battery
- added C1, C2: 10 uF, symbol Device:C
- added C3, C4: 22 uF, symbol Device:C
- added D1: APA-106-F5, LED_THT:LED_D5.0mm-4_RGB, symbol LED:APA-106-F5
- added H1, H2, H3, H4, H5, H6, H7, H8: MountingHole, MountingHole:MountingHole_3.5mm, symbol Mechanical:MountingHole
- added J2: Conn_01x08_Pin, Connector_PinHeader_1.00mm:PinHeader_1x08_P1.00mm_Vertical, symbol Connector:Conn_01x08_Pin
- added R1, R2, R3: 220, Resistor_THT:R_Axial_DIN0204_L3.6mm_D1.6mm_P5.08mm_Horizontal, symbol Device:R
- added U10, U9: Bidirectional ESC, Bidirectional_ESC:Bi_ESC_foot, symbol Brushed ESC:Brushed_ESC
- U1: value E -> Rasberry Pi 0W
- U8: footprint (none) -> Flysky fs-a8s:Flysky fs-a8s_footprint
Connections:
- net +3.3V: now also J2.7 (Pin_7)
- net +5V: now also U1.2 (5V_2), J2.2 (Pin_2)
- net 0: now also U1.6 (GND_6), U6.5 (IN-), U7.5 (IN-), BT1.2 (-), D1.2 (GND), J2.1 (Pin_1), J2.8 (Pin_8), U10.6 (B1_-), U9.6 (B1_-)
- net at U6.2 (OUT+): now also C3.1
- net at U6.3 (OUT-): now also C3.2
- net at U6.6 (IN-): now also C1.2
- net at U6.7 (IN+): now also C1.1
- net +7.5V: now reaches U6.8 (IN+)
- net +7.5V: now also U7.8 (IN+), BT1.1 (+), U10.5 (B1_+), U9.5 (B1_+)
- net at U7.2 (OUT+): now also C4.2
- net at U7.3 (OUT-): now also C4.1
- net at U7.6 (IN-): now also C2.1
- net at U7.7 (IN+): now also C2.2
- net at J1.10 (Pin_10): now also U10.7 (S1)
- net at J1.11 (Pin_11): now also U10.10 (S2)
- net at J1.18 (Pin_18): now also U9.7 (S1)
- net at J1.19 (Pin_19): now also U9.10 (S2)
- net at J1.20 (Pin_20): now also J2.3 (Pin_3)
- net at J1.22 (Pin_22): now also J2.4 (Pin_4)
- net at J1.23 (Pin_23): now also J2.5 (Pin_5)
- net at J1.24 (Pin_24): now also J2.6 (Pin_6)
- net at J1.6 (Pin_6): now also R3.2
- net at J1.7 (Pin_7): now also R2.2
- net at J1.8 (Pin_8): now also R1.2
- new net: D1.1 (DO), R1.1
- new net: D1.3 (VDD), R2.1
- new net: D1.4 (DI), R3.1
- no-connect marks 5 -> 63
Other:
- moved on the sheet: J1, U1

Commit message: welcome
Parts:
- removed U10, U9: Bidirectional ESC, Bidirectional_ESC:Bi_ESC_foot, symbol Brushed ESC:Brushed_ESC
- added U10: ~, 4x1_ESC:4x1_ESC, symbol 4x1_ESC:4x1_ESC
Connections:
- net +7.5V: now also U10.14 (BT1)
- net at J1.11 (Pin_11): now also U10.5 (PWM3)
- net at J1.10 (Pin_10): now also U10.4 (PWM2)
- net at J1.12 (Pin_12): now also U10.6 (PWM4)
- net at J1.9 (Pin_9): now also U10.3 (PWM1)
- new net GND: U10.1 (GND), U10.13 (GND)
- no-connect marks 63 -> 64
Other:
- moved on the sheet: H1, H2, H3, H4, H5, H6, H7, H8
