File: NEW/Drone_1.kicad_pcb (KiCad board)
At the start: 4 copper layers, 100 x 120 mm, 25 parts, among them J1 ESP-32_DevkitC, J2 Conn_01x08_Pin, U1 Rasberry Pi 0W, U10 Bidirectional ESC, U2 MPU6050, U3 GY-NEO6MV2, U4 BME280, U5 HMC5883L, U6 mp1584, U7 mp1584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

Commit message: welcome
Routing:
- net 0: track 0.00 -> 41.2 mm, vias 0 -> 7
- net +5V: track 0.00 -> 6.77 mm, vias 0 -> 2
- net +7.5V: track 0.00 -> 4.77 mm, vias 0 -> 2
- added copper zone on In1.Cu, net +3.3V
- added copper zone on In1.Cu, net +5V
- added copper zone on In2.Cu, net +7.5V
- added copper zone on B.Cu, net 0

Commit message: welcome
Parts:
- moved J2 0.91 mm to (66.4, 109.7)
- moved U2 0.69 mm to (137.5, 72.4)
Routing:
- net Net-(J1-Pin_29): track 40.6 -> 48.8 mm
- net Net-(J1-Pin_30): track 50.2 -> 45.3 mm
- net 0: track 41.2 -> 43.0 mm
- net Net-(J1-Pin_20): track 73.7 -> 74.7 mm
- net Net-(J1-Pin_23): track 64.6 -> 65.4 mm
- net Net-(J1-Pin_24): track 62.4 -> 63.2 mm
- net Net-(J1-Pin_22): track 66.8 -> 67.7 mm
- net +5V: track 6.77 -> 7.48 mm
- net +7.5V: track 4.77 -> 5.37 mm

Commit message: welcome
Parts:
- removed U9: Bidirectional ESC, Bidirectional_ESC:Bi_ESC_foot
- U10: value Bidirectional ESC -> ~; footprint Bidirectional_ESC:Bi_ESC_foot -> 4x1_ESC:4x1_ESC
- moved U10 93.3 mm to (149.1, 89.8)
Connections:
- J1 pad 12: unconnected-(J1-Pin_12-Pad12) -> Net-(J1-Pin_12)
- J1 pad 18: Net-(J1-Pin_18) -> unconnected-(J1-Pin_18-Pad18)
- J1 pad 19: Net-(J1-Pin_19) -> unconnected-(J1-Pin_19-Pad19)
- J1 pad 9: unconnected-(J1-Pin_9-Pad9) -> Net-(J1-Pin_9)
Routing:
- net Net-(J1-Pin_10): track 113.8 -> 0.00 mm
- net Net-(J1-Pin_11): track 110.4 -> 0.00 mm
- net Net-(J1-Pin_19): track 25.0 -> 0.00 mm
- net Net-(J1-Pin_18): track 21.6 -> 0.00 mm
- net 0: track 43.0 -> 24.4 mm, vias 7 -> 5
- net +7.5V: track 5.37 -> 17.1 mm
- net GND: track 0.00 -> 11.6 mm, vias 0 -> 1
- net Net-(J1-Pin_21): track 32.3 -> 26.5 mm
- net Net-(J1-Pin_28): track 41.4 -> 39.5 mm
- net Net-(J1-Pin_24): track 63.2 -> 62.7 mm

Commit message: welcome
Parts:
- removed U2: MPU6050, MPU6050_footprint:MPU6050foot
- added U9: ~, MPU6500:MPU6500, F.Cu at (145.8, 85.7)
- moved U10 13.9 mm to (159.6, 99.0)
- moved U8 1.17 mm to (120.8, 92.4)
Connections:
- J1 pad 25: unconnected-(J1-Pin_25-Pad25) -> Net-(J1-Pin_25)
- J1 pad 26: unconnected-(J1-Pin_26-Pad26) -> Net-(J1-Pin_26)
- J2 pad 6: Net-(J1-Pin_24) -> Net-(J1-Pin_29)
- U10 pad 13: GND -> 0
Routing:
- net Net-(J1-Pin_12): track 0.00 -> 54.0 mm
- net Net-(J1-Pin_26): track 0.00 -> 53.2 mm
- net Net-(J1-Pin_11): track 0.00 -> 52.0 mm
- net Net-(J1-Pin_10): track 0.00 -> 50.5 mm
- net Net-(J1-Pin_9): track 0.00 -> 47.9 mm
- net Net-(J1-Pin_25): track 0.00 -> 42.7 mm
- net Net-(J1-Pin_24): track 62.7 -> 28.0 mm
- net 0: track 24.4 -> 46.4 mm, vias 5 -> 7
- net +7.5V: track 17.1 -> 3.40 mm, vias 2 -> 1
- net Net-(J1-Pin_30): track 44.8 -> 56.9 mm
- net GND: track 11.6 -> 0.00 mm, vias 1 -> 0
- net Net-(J1-Pin_21): track 26.5 -> 19.0 mm
- net +5V: track 7.48 -> 9.73 mm

Commit message: welcome
Connections:
- J1 pad 14: 0 -> unconnected-(J1-Pin_14-Pad14)
- J1 pad 15: +3.3V -> unconnected-(J1-Pin_15-Pad15)
- J1 pad 16: unconnected-(J1-Pin_16-Pad16) -> +3.3V
- J1 pad 17: unconnected-(J1-Pin_17-Pad17) -> 0
- U1 pad 10: unconnected-(U1-GPIO15/RXD0-Pad10) -> Net-(J1-Pin_28)
- U1 pad 8: unconnected-(U1-GPIO14/TXD0-Pad8) -> Net-(J1-Pin_27)
Routing:
- net Net-(J1-Pin_28): track 39.5 -> 72.6 mm
- net Net-(J1-Pin_27): track 43.9 -> 62.0 mm

Commit message: welcome
Parts:
- moved U10 98.9 mm to (60.8, 96.4), turned to -90 degrees
- moved J2 90.3 mm to (156.5, 103.0)
- moved U3 2.11 mm to (84.7, 100.0)
- moved U1 1.27 mm to (112.2, 67.5)
- moved U8 1.20 mm to (121.7, 91.6)
- moved U4 0.41 mm to (79.7, 126.2)
Connections:
- J1 pad 18: unconnected-(J1-Pin_18-Pad18) -> Net-(J1-Pin_18)
- J1 pad 19: unconnected-(J1-Pin_19-Pad19) -> Net-(J1-Pin_19)
- J1 pad 29: Net-(J1-Pin_29) -> unconnected-(J1-Pin_29-Pad29)
- J2 pad 2: +5V -> +3.3V
- J2 pad 3: Net-(J1-Pin_20) -> Net-(J1-Pin_18)
- J2 pad 4: Net-(J1-Pin_22) -> Net-(J1-Pin_19)
- J2 pad 5: Net-(J1-Pin_23) -> Net-(J1-Pin_20)
- J2 pad 6: Net-(J1-Pin_29) -> Net-(J1-Pin_23)
- J2 pad 7: +3.3V -> +5V
- U10 pad 3: Net-(J1-Pin_9) -> Net-(J1-Pin_12)
- U10 pad 4: Net-(J1-Pin_10) -> Net-(J1-Pin_11)
- U10 pad 5: Net-(J1-Pin_11) -> Net-(J1-Pin_10)
- U10 pad 6: Net-(J1-Pin_12) -> Net-(J1-Pin_9)
- U3 pad 2: Net-(J1-Pin_27) -> Net-(J1-Pin_22)
- U3 pad 3: Net-(J1-Pin_28) -> Net-(J1-Pin_21)
Routing:
- net Net-(J1-Pin_21): track 19.0 -> 79.2 mm
- net Net-(J1-Pin_20): track 74.7 -> 22.1 mm
- net Net-(J1-Pin_29): track 49.1 -> 0.00 mm
- net Net-(J1-Pin_28): track 72.6 -> 35.7 mm
- net Net-(J1-Pin_23): track 65.4 -> 32.1 mm
- net Net-(J1-Pin_12): track 54.0 -> 86.4 mm
- net Net-(J1-Pin_11): track 52.0 -> 83.1 mm
- net Net-(J1-Pin_10): track 50.5 -> 80.0 mm
- net Net-(J1-Pin_9): track 47.9 -> 75.5 mm
- net 0: track 46.4 -> 21.2 mm, vias 7 -> 4
- net Net-(J1-Pin_27): track 62.0 -> 41.7 mm
- net Net-(J1-Pin_19): track 0.00 -> 19.2 mm
- net Net-(J1-Pin_18): track 0.00 -> 16.2 mm
- net Net-(J1-Pin_22): track 67.7 -> 52.0 mm
- net +7.5V: track 3.40 -> 10.7 mm
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
Commit message: welcome
Parts:
- added G***: LOGO, Graphics:biggerdrone, F.Cu at (137.2, 55.6)
- added G***: LOGO, Graphics:words, F.Cu at (137.4, 65.9)
- added R4: 3.3K, Resistor_THT:R_Axial_DIN0204_L3.6mm_D1.6mm_P5.08mm_Horizontal, F.Cu at (157.5, 89.3)
- added R5: 2K, Resistor_THT:R_Axial_DIN0204_L3.6mm_D1.6mm_P5.08mm_Horizontal, F.Cu at (157.5, 79.1)
- moved BT1 85.5 mm to (152.8, 68.0), turned to -90 degrees
- moved U6 81.6 mm to (69.7, 61.9), turned to 90 degrees
- moved U7 73.8 mm to (138.4, 88.9)
- moved U9 43.3 mm to (115.2, 116.3)
- moved R3 26.3 mm to (100.8, 145.1), turned to 180 degrees
- moved R2 17.1 mm to (110.3, 145.1), turned to 180 degrees
- moved U4 13.1 mm to (67.6, 131.2), turned to 90 degrees
- moved U3 11.6 mm to (84.5, 111.6)
- moved J1 10.3 mm to (107.0, 137.1)
- moved R1 9.01 mm to (120.0, 145.1), turned to 180 degrees
- moved U8 8.16 mm to (122.0, 83.5)
- moved U5 7.03 mm to (92.3, 142.5)
- moved U1 3.71 mm to (111.8, 63.8)
- moved D1 3.20 mm to (127.7, 142.7)
- moved J2 1.60 mm to (154.9, 103.1)
Connections:
- J1 pad 13: unconnected-(J1-Pin_13-Pad13) -> Net-(J1-Pin_13)
- J1 pad 14: unconnected-(J1-Pin_14-Pad14) -> 0
- J1 pad 15: unconnected-(J1-Pin_15-Pad15) -> +3.3V
- J1 pad 16: +3.3V -> unconnected-(J1-Pin_16-Pad16)
- J1 pad 17: 0 -> unconnected-(J1-Pin_17-Pad17)
- U3 pad 2: Net-(J1-Pin_22) -> Net-(J1-Pin_21)
- U3 pad 3: Net-(J1-Pin_21) -> Net-(J1-Pin_22)
- U8 pad 1: 0 -> Net-(U8-GND)
- U8 pad 3: Net-(J1-Pin_21) -> Net-(U8-SBUS)
Routing:
- net Net-(J1-Pin_13): track 0.00 -> 56.1 mm
- net Net-(J1-Pin_30): track 56.9 -> 3.27 mm
- net Net-(J1-Pin_26): track 53.2 -> 3.27 mm
- net Net-(J1-Pin_25): track 42.7 -> 3.27 mm
- net Net-(J1-Pin_28): track 35.7 -> 64.3 mm
- net Net-(J1-Pin_6): track 7.89 -> 27.3 mm
- net Net-(J1-Pin_4): track 39.8 -> 21.7 mm
- net 0: track 21.2 -> 5.36 mm, vias 4 -> 1
- net Net-(J1-Pin_27): track 41.7 -> 55.6 mm
- net Net-(D1-DI): track 19.1 -> 28.8 mm
- net Net-(J1-Pin_7): track 11.3 -> 20.3 mm
- net Net-(J1-Pin_21): track 79.2 -> 70.6 mm
- net Net-(J1-Pin_19): track 19.2 -> 25.8 mm
- net Net-(J1-Pin_18): track 16.2 -> 22.9 mm
- net Net-(J1-Pin_20): track 22.1 -> 28.8 mm
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