File: NEW/Drone_1.kicad_sch (KiCad schematic)
At the start: 29 parts, among them J1 ESP-32_DevkitC, J2 Conn_01x08_Pin, U1 Rasberry Pi 0W, U10 Bidirectional ESC, U2 MPU6050, U3 GY-NEO6MV2, U4 BME280, U5 HMC5883L, U6 mp1584, U7 mp1584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

Commit message: welcome
Parts:
- removed U10, U9: Bidirectional ESC, Bidirectional_ESC:Bi_ESC_foot, symbol Brushed ESC:Brushed_ESC
- added U10: ~, 4x1_ESC:4x1_ESC, symbol 4x1_ESC:4x1_ESC
Connections:
- net +7.5V: now also U10.14 (BT1)
- net at J1.11 (Pin_11): now also U10.5 (PWM3)
- net at J1.10 (Pin_10): now also U10.4 (PWM2)
- net at J1.12 (Pin_12): now also U10.6 (PWM4)
- net at J1.9 (Pin_9): now also U10.3 (PWM1)
- new net GND: U10.1 (GND), U10.13 (GND)
- no-connect marks 63 -> 64
Other:
- moved on the sheet: H1, H2, H3, H4, H5, H6, H7, H8

Commit message: welcome
Parts:
- added U9: ~, symbol MPU6500:MPU6500m
Connections:
- net GND is gone; now on net 0: U10.1 (GND), U10.13 (GND)

Commit message: welcome
Parts:
- removed U2: MPU6050, MPU6050_footprint:MPU6050foot, symbol MPU6050_module:MPU6050m
- U9: footprint (none) -> MPU6500:MPU6500
Connections:
- net +3.3V: now also U9.1 (VCC)
- net 0: now also U9.2 (GND)
- net at J1.29 (Pin_29): now also J2.6 (Pin_6)
- net at J1.30 (Pin_30): now also U9.4 (SDA)
- net at J1.24 (Pin_24): now also U9.3 (SCL); no longer J2.6 (Pin_6)
- net at U9.8 (INT): now also J1.26 (Pin_26)
- net at U9.9 (NCS): now also J1.25 (Pin_25)
- no-connect marks 64 -> 63
Other:
- moved on the sheet: U3, U9

Commit message: welcome
Connections:
- net +3.3V: now also J1.16 (Pin_16); no longer J1.15 (Pin_15)
- net 0: now also J1.17 (Pin_17); no longer J1.14 (Pin_14)
- net at J1.27 (Pin_27), U3.2 (RX): now also U1.8 (GPIO14/TXD0)
- net at J1.28 (Pin_28), U3.3 (TX): now also U1.10 (GPIO15/RXD0)
- no-connect marks 63 -> 61

Commit message: welcome
Connections:
- net +3.3V: now also J2.2 (Pin_2); no longer J2.7 (Pin_7)
- net +5V: now also J2.7 (Pin_7); no longer J2.2 (Pin_2)
- net at J2.3 (Pin_3): now also J1.18 (Pin_18); no longer J1.20 (Pin_20)
- net at J2.4 (Pin_4): now also J1.19 (Pin_19); no longer J1.22 (Pin_22)
- net at J2.5 (Pin_5): now also J1.20 (Pin_20); no longer J1.23 (Pin_23)
- net at J2.6 (Pin_6): now also J1.23 (Pin_23); no longer J1.29 (Pin_29)
- net at J1.10 (Pin_10): now also U10.5 (PWM3); no longer U10.4 (PWM2)
- net at J1.11 (Pin_11): now also U10.4 (PWM2); no longer U10.5 (PWM3)
- net at J1.12 (Pin_12): now also U10.3 (PWM1); no longer U10.6 (PWM4)
- net at J1.21 (Pin_21), U8.3 (SBUS): now also U3.3 (TX)
- net at J1.27 (Pin_27), U1.8 (GPIO14/TXD0): no longer U3.2 (RX)
- net at J1.28 (Pin_28), U1.10 (GPIO15/RXD0): no longer U3.3 (TX)
- net at J1.9 (Pin_9): now also U10.6 (PWM4); no longer U10.3 (PWM1)
- new net: J1.22 (Pin_22), U3.2 (RX)
- no-connect marks 61 -> 60
Other:
- moved on the sheet: J2, U1, U10, U3

Commit message: welcome
Parts:
- added R4: 3.3K, Resistor_THT:R_Axial_DIN0204_L3.6mm_D1.6mm_P5.08mm_Horizontal, symbol Device:R
- added R5: 2K, Resistor_THT:R_Axial_DIN0204_L3.6mm_D1.6mm_P5.08mm_Horizontal, symbol Device:R
Connections:
- net +3.3V: now also J1.15 (Pin_15); no longer J1.16 (Pin_16)
- net 0: now also J1.14 (Pin_14), R5.1; no longer J1.17 (Pin_17), U8.1 (GND)
- net at J1.13 (Pin_13): now also R4.1
- net at U3.2 (RX): now also J1.21 (Pin_21); no longer J1.22 (Pin_22)
- new net: R5.2, U8.1 (GND)
- new net: J1.22 (Pin_22), U3.3 (TX)
- new net: R4.2, U8.3 (SBUS)
- no-connect marks 60 -> 59
